Commit message: Files converted from MuJoCo models

File: urdf/iiwa14/iiwa14.urdf (robot description, URDF)
Before this commit: robot iiwa14, 17 links, 16 joints
Links:
- link base: geometry visual mesh filename=package://serial_link_velocity_control/urdf/iiwa14/link_0.s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
- link link1: geometry visual mesh filename=package://serial_link_velocity_control/urdf/iiwa14/link_1.s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
- link link2: geometry visual mesh filename=package://serial_link_velocity_control/urdf/iiwa14/link_2_g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; visual mesh filename=package://serial_link_velocity_control/urdf/iiwa14/link_2_o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
- link link3: geometry visual mesh filename=package://serial_link_velocity_control/urdf/iiwa14/band.stl; visual mesh filename=package://serial_link_velocity_control/urdf/iiwa14/kuka.stl
- link link4: geometry visual mesh filename=package://serial_link_velocity_control/urdf/iiwa14/link_4_g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; visual mesh filename=package://serial_link_velocity_control/urdf/iiwa14/link_4_o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
- link link5: geometry visual mesh filename=package://serial_link_velocity_control/urdf/iiwa14/band.stl; visual mesh filename=package://serial_link_velocity_control/urdf/iiwa14/kuka.stl
- link link6: geometry visual mesh filename=package://serial_link_velocity_control/urdf/iiwa14/link_6_g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; visual mesh filename=package://serial_link_velocity_control/urdf/iiwa14/link_6_o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
- link link7: geometry visual mesh filename=package://serial_link_velocity_control/urdf/iiwa14/link_7.s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
